Commit message: introduce origin as parameter for multirotor_base_macro so that one can set offset between base_link and base_link_inertia from <drones>.xacro files

File: rotors_gazebo/models/rotors_description/urdf/multirotor_base.xacro (robot description, xacro)
@@ -19,8 +19,8 @@
   <!-- Main multirotor link -->
   <xacro:macro name="multirotor_base_macro"
-    params="robot_namespace mass body_width body_height mesh_file mesh_scale color *inertia">
+    params="robot_namespace mass body_width body_height mesh_file mesh_scale color *inertia *origin">
     <link name="base_link"></link>
     <joint name="base_joint" type="fixed">
-      <origin xyz="0 0 0" rpy="0 0 0" />
+      <xacro:insert_block name="origin"/>
       <parent link="base_link" />
       <child link="base_link_inertia" />
